File: hardware/conductivity/conductivity.sch (EAGLE design)
At the start: 18 parts, among them IC1 AD820R, U1 TLV2374IDR, U2 TLE2426CD

Commit message: board and parts list update june 2018
Parts:
- D1, D2: device fab:DIODESOD123 -> trellisLaura:DIODESOD123
Connections:
- net FROMWATER: now also SV1.6; no longer SV1.5
- net N$13: now also SV1.4; no longer SV1.6
- net N$16: now also SV1.5; no longer SV1.4
Other:
- moved on the sheet: D2, R9, SV1
Changed lines of the file:
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@@
 <?xml version="1.0" encoding="utf-8"?>
 <!DOCTYPE eagle SYSTEM "eagle.dtd">
-<eagle version="6.2">
+<eagle version="8.6.3">
 <drawing>
 <settings>
 <setting alwaysvectorfont="no"/>
+<setting keepoldvectorfont="yes"/>
 <setting verticaltext="up"/>
 </settings>
-<grid distance="0.1" unitdist="inch" unit="inch" style="lines" multiple="1" display="no" altdistance="0.01" altunitdist="inch" altunit="inch"/>
+<grid distance="0.05" unitdist="inch" unit="inch" style="lines" multiple="1" display="no" altdistance="0.01" altunitdist="inch" altunit="inch"/>
 <layers>
 <layer number="1" name="Top" color="4" fill="1" visible="no" active="no"/>
@@
 <layer number="59" name="tCarbon" color="7" fill="1" visible="no" active="no"/>
 <layer number="60" name="bCarbon" color="7" fill="1" visible="no" active="no"/>
+<layer number="88" name="SimResults" color="9" fill="1" visible="yes" active="yes"/>
+<layer number="89" name="SimProbes" color="9" fill="1" visible="yes" active="yes"/>
 <layer number="90" name="Modules" color="5" fill="1" visible="yes" active="yes"/>
 <layer number="91" name="Nets" color="2" fill="1" visible="yes" active="yes"/>
@@
 <layer number="230" name="230bmp" color="7" fill="1" visible="yes" active="yes"/>
 <layer number="231" name="231bmp" color="7" fill="1" visible="yes" active="yes"/>
+<layer number="232" name="Eagle3D_PG2" color="7" fill="1" visible="no" active="no"/>
+<layer number="233" name="Eagle3D_PG3" color="7" fill="1" visible="no" active="no"/>
 <layer number="248" name="Housing" color="7" fill="1" visible="yes" active="yes"/>
 <layer number="249" name="Edge" color="7" fill="1" visible="yes" active="yes"/>
@@
 <part name="R9" library="SparkFun-Resistors" deviceset="4.7KOHM" device="-0603-1/10W-1%" value="4.7k"/>
 <part name="R10" library="SparkFun-Resistors" deviceset="1.20KOHM" device="-0603-1/10W-1%" value="1.20k"/>
-<part name="D1" library="fab" deviceset="DIODE" device="SOD123"/>
-<part name="D2" library="fab" deviceset="DIODE" device="SOD123"/>
+<part name="D1" library="trellisLaura" deviceset="DIODE" device="SOD123"/>
+<part name="D2" library="trellisLaura" deviceset="DIODE" device="SOD123"/>
 <part name="C2" library="SparkFun-Capacitors" deviceset="0.1UF" device="-0603-25V-5%" value="0.1uF"/>
 <part name="U2" library="TLE2426CD" deviceset="TLE2426CD" device=""/>
@@
 <instance part="R5" gate="G$1" x="175.26" y="137.16"/>
 <instance part="R8" gate="G$1" x="154.94" y="83.82" rot="R90"/>
-<instance part="R9" gate="G$1" x="106.68" y="142.24"/>
+<instance part="R9" gate="G$1" x="104.14" y="151.13"/>
 <instance part="R10" gate="G$1" x="99.06" y="124.46" rot="R90"/>
 <instance part="D1" gate="G$1" x="137.16" y="152.4"/>
-<instance part="D2" gate="G$1" x="144.78" y="139.7" rot="R180"/>
+<instance part="D2" gate="G$1" x="143.51" y="139.7" rot="R180"/>
 <instance part="C2" gate="G$1" x="190.5" y="137.16" rot="R90"/>
 <instance part="U2" gate="A" x="60.96" y="86.36"/>
 <instance part="S1" gate="1" x="101.6" y="114.3" rot="R90"/>
 <instance part="R7" gate="G$1" x="109.22" y="124.46" rot="R90"/>
-<instance part="SV1" gate="1" x="111.76" y="33.02" rot="R90"/>
+<instance part="SV1" gate="1" x="111.76" y="21.59" rot="R90"/>
 </instances>
 <busses>
@@
 <junction x="88.9" y="111.76"/>
 <wire x1="88.9" y1="104.14" x2="109.22" y2="104.14" width="0.1524" layer="91"/>
-<wire x1="109.22" y1="104.14" x2="109.22" y2="40.64" width="0.1524" layer="91"/>
+<wire x1="109.22" y1="104.14" x2="109.22" y2="45.72" width="0.1524" layer="91"/>
 <pinref part="S1" gate="1" pin="P"/>
-<pinref part="SV1" gate="1" pin="5"/>
+<pinref part="SV1" gate="1" pin="6"/>
+<wire x1="109.22" y1="45.72" x2="106.68" y2="45.72" width="0.1524" layer="91"/>
+<wire x1="106.68" y1="45.72" x2="106.68" y2="29.21" width="0.1524" layer="91"/>
 </segment>
 </net>
@@
 <wire x1="86.36" y1="142.24" x2="93.98" y2="142.24" width="0.1524" layer="91"/>
 <pinref part="R10" gate="G$1" pin="2"/>
-<wire x1="93.98" y1="142.24" x2="101.6" y2="142.24" width="0.1524" layer="91"/>
+<wire x1="93.98" y1="142.24" x2="99.06" y2="151.13" width="0.1524" layer="91"/>
 <wire x1="99.06" y1="129.54" x2="93.98" y2="129.54" width="0.1524" layer="91"/>
 <wire x1="93.98" y1="129.54" x2="93.98" y2="142.24" width="0.1524" layer="91"/>
@@
 <pinref part="R7" gate="G$1" pin="2"/>
 <wire x1="109.22" y1="129.54" x2="101.6" y2="129.54" width="0.1524" layer="91"/>
-<wire x1="101.6" y1="129.54" x2="101.6" y2="142.24" width="0.1524" layer="91"/>
+<wire x1="101.6" y1="129.54" x2="99.06" y2="151.13" width="0.1524" layer="91"/>
 <pinref part="R9" gate="G$1" pin="1"/>
-<junction x="101.6" y="142.24"/>
+<junction x="99.06" y="151.13"/>
 </segment>
 </net>
@@
 <segment>
 <pinref part="U1" gate="A" pin="2IN-"/>
-<wire x1="111.76" y1="142.24" x2="116.84" y2="142.24" width="0.1524" layer="91"/>
+<wire x1="109.22" y1="151.13" x2="116.84" y2="142.24" width="0.1524" layer="91"/>
 <wire x1="116.84" y1="142.24" x2="124.46" y2="142.24" width="0.1524" layer="91"/>
 <wire x1="124.46" y1="142.24" x2="160.02" y2="142.24" width="0.1524" layer="91"/>
@@
 <wire x1="149.86" y1="152.4" x2="149.86" y2="139.7" width="0.1524" layer="91"/>
 <wire x1="149.86" y1="139.7" x2="149.86" y2="134.62" width="0.1524" layer="91"/>
-<wire x1="149.86" y1="139.7" x2="147.32" y2="139.7" width="0.1524" layer="91"/>
+<wire x1="149.86" y1="139.7" x2="146.05" y2="139.7" width="0.1524" layer="91"/>
 <junction x="149.86" y="139.7"/>
 <pinref part="D2" gate="G$1" pin="A"/>
@@
 <pinref part="D2" gate="G$1" pin="C"/>
 <pinref part="R1" gate="G$1" pin="2"/>
-<wire x1="142.24" y1="139.7" x2="127" y2="139.7" width="0.1524" layer="91"/>
-<wire x1="142.24" y1="139.7" x2="142.24" y2="91.44" width="0.1524" layer="91"/>
+<wire x1="140.97" y1="139.7" x2="127" y2="139.7" width="0.1524" layer="91"/>
+<wire x1="140.97" y1="139.7" x2="142.24" y2="91.44" width="0.1524" layer="91"/>
 <wire x1="142.24" y1="91.44" x2="162.56" y2="91.44" width="0.1524" layer="91"/>
 <pinref part="U1" gate="A" pin="3IN+"/>
 <wire x1="162.56" y1="91.44" x2="162.56" y2="99.06" width="0.1524" layer="91"/>
+<junction x="140.97" y="139.7"/>
 </segment>
 </net>
@@
 <net name="N$13" class="0">
 <segment>
-<pinref part="SV1" gate="1" pin="6"/>
 <wire x1="198.12" y1="96.52" x2="198.12" y2="48.26" width="0.1524" layer="91"/>
-<wire x1="198.12" y1="48.26" x2="106.68" y2="48.26" width="0.1524" layer="91"/>
-<wire x1="106.68" y1="48.26" x2="106.68" y2="40.64" width="0.1524" layer="91"/>
+<wire x1="198.12" y1="48.26" x2="113.03" y2="48.26" width="0.1524" layer="91"/>
 <pinref part="U1" gate="A" pin="4IN-"/>
 <wire x1="170.18" y1="99.06" x2="170.18" y2="96.52" width="0.1524" layer="91"/>
@@
 <wire x1="154.94" y1="134.62" x2="198.12" y2="134.62" width="0.1524" layer="91"/>
 <wire x1="198.12" y1="134.62" x2="198.12" y2="96.52" width="0.1524" layer="91"/>
+<pinref part="SV1" gate="1" pin="4"/>
+<junction x="111.76" y="29.21"/>
+<wire x1="111.76" y1="29.21" x2="111.76" y2="41.91" width="0.1524" layer="91"/>
+<wire x1="111.76" y1="41.91" x2="113.03" y2="41.91" width="0.1524" layer="91"/>
+<wire x1="113.03" y1="48.26" x2="113.03" y2="41.91" width="0.1524" layer="91"/>
 </segment>
 </net>
@@
 <net name="N$14" class="0">
 <segment>
-<wire x1="116.84" y1="45.72" x2="116.84" y2="40.64" width="0.1524" layer="91"/>
+<wire x1="116.84" y1="45.72" x2="116.84" y2="29.21" width="0.1524" layer="91"/>
 <pinref part="R8" gate="G$1" pin="1"/>
 <wire x1="116.84" y1="45.72" x2="154.94" y2="45.72" width="0.1524" layer="91"/>
@@
 <net name="N$16" class="0">
 <segment>
-<wire x1="111.76" y1="40.64" x2="111.76" y2="162.56" width="0.1524" layer="91"/>
 <pinref part="R6" gate="G$1" pin="2"/>
 <pinref part="U1" gate="A" pin="1OUT"/>
+<wire x1="111.76" y1="43.18" x2="111.76" y2="162.56" width="0.1524" layer="91"/>
 <wire x1="134.62" y1="134.62" x2="147.32" y2="134.62" width="0.1524" layer="91"/>
 <junction x="147.32" y="134.62"/>
 <wire x1="147.32" y1="134.62" x2="147.32" y2="162.56" width="0.1524" layer="91"/>
 <wire x1="111.76" y1="162.56" x2="147.32" y2="162.56" width="0.1524" layer="91"/>
-<pinref part="SV1" gate="1" pin="4"/>
+<pinref part="SV1" gate="1" pin="5"/>
+<wire x1="111.76" y1="43.18" x2="109.22" y2="43.18" width="0.1524" layer="91"/>
+<wire x1="109.22" y1="43.18" x2="109.22" y2="29.21" width="0.1524" layer="91"/>
 </segment>
 </net>
@@
 <pinref part="U2" gate="A" pin="IN"/>
 <wire x1="30.48" y1="93.98" x2="38.1" y2="93.98" width="0.1524" layer="91"/>
-<wire x1="119.38" y1="40.64" x2="119.38" y2="50.8" width="0.1524" layer="91"/>
+<wire x1="119.38" y1="29.21" x2="119.38" y2="50.8" width="0.1524" layer="91"/>
 <junction x="119.38" y="50.8"/>
 <pinref part="SV1" gate="1" pin="1"/>
+<junction x="81.28" y="50.8"/>
 </segment>
 </net>
 <net name="N$15" class="0">
 <segment>
-<wire x1="114.3" y1="40.64" x2="114.3" y2="60.96" width="0.1524" layer="91"/>
+<wire x1="114.3" y1="29.21" x2="114.3" y2="60.96" width="0.1524" layer="91"/>
 <wire x1="114.3" y1="60.96" x2="175.26" y2="60.96" width="0.1524" layer="91"/>
 <wire x1="175.26" y1="60.96" x2="175.26" y2="99.06" width="0.1524" layer="91"/>

Commit message: november update
Parts:
- removed SV1: (no value), con-lstb:MA06-1
- added JP1: (no value), pinhead:PINHD-1X2
- added JP2: (no value), pinhead:PINHD-1X4
Connections:
- net FROMWATER: now also JP1.2; no longer SV1.6
- net N$1: now also JP2.1; no longer SV1.1
- net N$13: now also JP2.4; no longer SV1.4
- net N$14: now also JP2.2; no longer SV1.2
- net N$15: now also JP2.3; no longer SV1.3
- net N$16: now also JP1.1; no longer SV1.5

Commit message: Revert "Updating."
Parts:
- removed JP1: (no value), pinhead:PINHD-1X2
- removed JP2: (no value), pinhead:PINHD-1X4
- added SV1: (no value), con-lstb:MA06-1
Connections:
- net FROMWATER: now also SV1.6; no longer JP1.2
- net N$1: now also SV1.1; no longer JP2.1
- net N$13: now also SV1.4; no longer JP2.4
- net N$14: now also SV1.2; no longer JP2.2
- net N$15: now also SV1.3; no longer JP2.3
- net N$16: now also SV1.5; no longer JP1.1
